File: hardware/ESP32_CP400/esp32_cp400.kicad_pcb (KiCad board)
At the start: 2 copper layers, 100 x 100 mm, 20 parts, among them J2 USB_A, J3 USB_A, J4 USB_A, J5 Micro_SD_Card, J6 Barrel_Jack, J7 DA15_Pins

Commit message: Add lock files for KiCad project with user information
- Created lock files for the KiCad PCB, project, and schematic for the ESP32_CP400 hardware.
- Each lock file contains the hostname and username for the user "Pedro".
Parts:
- added G***: LOGO, TRH:TRH_NEW, F.Cu at (123.5, 66.9)
- added kibuzzard-6A32A222: G***, kibuzzard-6A32A222, F.Cu at (145.0, 69.1)
- added kibuzzard-6A32A22E: G***, kibuzzard-6A32A22E, F.Cu at (139.3, 66.8)
- added kibuzzard-6A32A25A: G***, kibuzzard-6A32A25A, F.Cu at (139.4, 63.7)
- R1, R2, R3, R4, R5, R6: moved to B.Cu
- moved J5 119.6 mm to (93.3, 95.0), turned to -90 degrees
- moved R6 112.7 mm to (186.8, 84.3), turned to 90 degrees
- moved R5 108.2 mm to (182.1, 84.3), turned to -90 degrees
- moved R4 103.8 mm to (177.3, 84.3), turned to 90 degrees
- moved J1 103.1 mm to (106.2, 113.6), turned to -90 degrees
- moved R3 99.6 mm to (172.6, 84.3), turned to -90 degrees
- moved R1 96.2 mm to (167.8, 84.3), turned to 90 degrees
- moved J8 94.9 mm to (116.6, 114.0), turned to 180 degrees
- moved R2 90.9 mm to (163.1, 84.3), turned to -90 degrees
- moved J3 76.6 mm to (137.1, 113.5), turned to 0 degrees
- moved J2 71.9 mm to (157.4, 113.5), turned to 0 degrees
- moved J6 70.7 mm to (109.0, 70.3), turned to -90 degrees
- moved J7 41.0 mm to (163.5, 67.0), turned to 180 degrees
- moved R9 40.0 mm to (112.5, 97.4), turned to 180 degrees
- moved R8 39.9 mm to (112.5, 94.0), turned to 180 degrees
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Routing:
- net +5V: track 0.00 -> 209.8 mm, vias 0 -> 2
- net +3.3V: track 0.00 -> 110.4 mm, vias 0 -> 2
- net Net-(J5-CMD): track 0.00 -> 75.7 mm, vias 0 -> 2
- net Net-(J5-CLK): track 0.00 -> 70.6 mm, vias 0 -> 2
- net Net-(J5-DAT0): track 0.00 -> 66.7 mm
- net Net-(U1-RST): track 0.00 -> 50.6 mm, vias 0 -> 2
- net Net-(F1-Pad2): track 0.00 -> 36.5 mm, vias 0 -> 2
- net Net-(U1-IO06): track 0.00 -> 35.9 mm, vias 0 -> 2
- net Net-(J3-D+): track 0.00 -> 32.3 mm
- net Net-(J3-D-): track 0.00 -> 31.7 mm
- net Net-(U1-IO04): track 0.00 -> 30.9 mm, vias 0 -> 2
- net Net-(U1-IO08): track 0.00 -> 29.5 mm, vias 0 -> 2
- net Net-(U1-IO07): track 0.00 -> 29.1 mm, vias 0 -> 2
- net Net-(J7-Pad3): track 0.00 -> 29.0 mm, vias 0 -> 2
- net Net-(U1-IO05): track 0.00 -> 24.7 mm, vias 0 -> 2
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- added copper zone on B.Cu, net GND
- added copper zone on F.Cu, net GND
Other:
- board size 100 x 100 mm -> 110 x 60 mm
