File: hardware/esp32_clones/esp32_clones.kicad_pcb (KiCad board)
At the start: 2 copper layers, 110 x 60 mm, 27 parts, among them J2 USB_A, J3 USB_A, J4 USB_A, J5 Micro_SD_Card, J6 Barrel_Jack, J7 DA15_Pins, J9 AudioJack2_Ground

Commit message: Add production files for ESP32 clone hardware
- Created BOM (bill of materials) file to list components and their specifications.
- Added designators file to map component designators to their respective quantities.
- Introduced IPC netlist file for electrical connections and layout.
- Included positions file to specify component placements on the PCB.
- Established symbol library table for component symbols used in the design.
Connections:
- J8 pad 1: Net-(U1-RST) -> unconnected-(J8-Pad1)
- J8 pad 2: GND -> Net-(U1-RST)
- J8 pad 3: unconnected-(J8-Pad3) -> GND
Routing:
- net Net-(U1-RST): track 48.2 -> 45.1 mm
Changed lines of the file:
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@@
 	(paper "A4")
 	(title_block
-		(title "ESP32-CP400")
-		(date "2026-06-18")
+		(title "ESP32 Clones")
+		(date "2026-08-02")
 		(rev "1.0")
 		(company "The Retro Hacker")
@@
 		(property ki_fp_filters "R_*")
 		(sheetname "/")
-		(sheetfile "esp32_cp400.kicad_sch")
+		(sheetfile "esp32_clones.kicad_sch")
 		(units
 			(unit
@@
 		(property ki_fp_filters "microSD*")
 		(sheetname "/")
-		(sheetfile "esp32_cp400.kicad_sch")
+		(sheetfile "esp32_clones.kicad_sch")
 		(units
 			(unit
@@
 		)
 		(sheetname "/")
-		(sheetfile "esp32_cp400.kicad_sch")
+		(sheetfile "esp32_clones.kicad_sch")
 		(units
 			(unit
@@
 		)
 		(sheetname "/")
-		(sheetfile "esp32_cp400.kicad_sch")
+		(sheetfile "esp32_clones.kicad_sch")
 		(units
 			(unit
@@
 			(layers "*.Cu" "*.Mask")
 			(remove_unused_layers no)
-			(net "Net-(U1-RST)")
+			(net "unconnected-(J8-Pad1)")
 			(pinfunction "1_1")
-			(pintype "input")
+			(pintype "input+no_connect")
 		)
 		(pad "2" thru_hole circle
@@
 			(layers "*.Cu" "*.Mask")
 			(remove_unused_layers no)
-			(net "GND")
+			(net "Net-(U1-RST)")
 			(pinfunction "2_2")
 			(pintype "input")
@@
 			(layers "*.Cu" "*.Mask")
 			(remove_unused_layers no)
-			(net "unconnected-(J8-Pad3)")
+			(net "GND")
 			(pinfunction "3_3")
-			(pintype "input+no_connect")
+			(pintype "input")
 		)
 		(pad "4" thru_hole circle
@@
 		)
 		(sheetname "/")
-		(sheetfile "esp32_cp400.kicad_sch")
+		(sheetfile "esp32_clones.kicad_sch")
 		(units
 			(unit
@@
 		(property ki_fp_filters "R_*")
 		(sheetname "/")
-		(sheetfile "esp32_cp400.kicad_sch")
+		(sheetfile "esp32_clones.kicad_sch")
 		(units
 			(unit
@@
 		(property ki_fp_filters "BarrelJack*")
 		(sheetname "/")
-		(sheetfile "esp32_cp400.kicad_sch")
+		(sheetfile "esp32_clones.kicad_sch")
 		(units
 			(unit
@@
 		(property ki_fp_filters "*Fuse*")
 		(sheetname "/")
-		(sheetfile "esp32_cp400.kicad_sch")
+		(sheetfile "esp32_clones.kicad_sch")
 		(units
 			(unit
@@
 		(property ki_fp_filters "Jack*")
 		(sheetname "/")
-		(sheetfile "esp32_cp400.kicad_sch")
+		(sheetfile "esp32_clones.kicad_sch")
 		(units
 			(unit
@@
 		(property ki_fp_filters "USB*")
 		(sheetname "/")
-		(sheetfile "esp32_cp400.kicad_sch")
+		(sheetfile "esp32_clones.kicad_sch")
 		(units
 			(unit
@@
 		(property ki_fp_filters "C_*")
 		(sheetname "/")
-		(sheetfile "esp32_cp400.kicad_sch")
+		(sheetfile "esp32_clones.kicad_sch")
 		(units
 			(unit
@@
 		(property ki_fp_filters "R_*")
 		(sheetname "/")
-		(sheetfile "esp32_cp400.kicad_sch")
+		(sheetfile "esp32_clones.kicad_sch")
 		(units
 			(unit
@@
 		(property ki_fp_filters "CP_*")
 		(sheetname "/")
-		(sheetfile "esp32_cp400.kicad_sch")
+		(sheetfile "esp32_clones.kicad_sch")
 		(units
 			(unit
@@
 		(property ki_fp_filters "DSUB*Pins*")
 		(sheetname "/")
-		(sheetfile "esp32_cp400.kicad_sch")
+		(sheetfile "esp32_clones.kicad_sch")
 		(units
 			(unit
@@
 		(property ki_fp_filters "USB*")
 		(sheetname "/")
-		(sheetfile "esp32_cp400.kicad_sch")
+		(sheetfile "esp32_clones.kicad_sch")
 		(units
 			(unit
@@
 		(property ki_fp_filters "R_*")
 		(sheetname "/")
-		(sheetfile "esp32_cp400.kicad_sch")
+		(sheetfile "esp32_clones.kicad_sch")
 		(units
 			(unit
@@
 		(property ki_fp_filters "USB*")
 		(sheetname "/")
-		(sheetfile "esp32_cp400.kicad_sch")
+		(sheetfile "esp32_clones.kicad_sch")
 		(units
 			(unit
@@
 		(property ki_fp_filters "R_*")
 		(sheetname "/")
-		(sheetfile "esp32_cp400.kicad_sch")
+		(sheetfile "esp32_clones.kicad_sch")
 		(units
 			(unit
@@
 		(property ki_fp_filters "R_*")
 		(sheetname "/")
-		(sheetfile "esp32_cp400.kicad_sch")
+		(sheetfile "esp32_clones.kicad_sch")
 		(units
 			(unit
@@
 		(property ki_fp_filters "R_*")
 		(sheetname "/")
-		(sheetfile "esp32_cp400.kicad_sch")
+		(sheetfile "esp32_clones.kicad_sch")
 		(units
 			(unit
@@
 		(property ki_fp_filters "R_*")
 		(sheetname "/")
-		(sheetfile "esp32_cp400.kicad_sch")
+		(sheetfile "esp32_clones.kicad_sch")
 		(units
 			(unit
@@
 		(property ki_fp_filters "R_*")
 		(sheetname "/")
-		(sheetfile "esp32_cp400.kicad_sch")
+		(sheetfile "esp32_clones.kicad_sch")
 		(units
 			(unit
@@
 		(property ki_fp_filters "R_*")
 		(sheetname "/")
-		(sheetfile "esp32_cp400.kicad_sch")
+		(sheetfile "esp32_clones.kicad_sch")
 		(units
 			(unit
@@
 	)
 	(segment
-		(start 121.55 113.325)
-		(end 121.55 100.9)
+		(start 118 111.825)
+		(end 119.975 111.825)
 		(width 0.2)
 		(layer "B.Cu")
@@
 	)
 	(segment
-		(start 118 115.025)
-		(end 119.85 115.025)
+		(start 121.55 110.25)
+		(end 121.55 100.9)
 		(width 0.2)
 		(layer "B.Cu")
@@
 	)
 	(segment
-		(start 121.55 100.9)
-		(end 124.125 98.325)
+		(start 148.685 99.035)
+		(end 148.685 102.075)
 		(width 0.2)
 		(layer "B.Cu")
@@
 	)
 	(segment
-		(start 148.685 99.035)
-		(end 148.685 102.075)
+		(start 119.975 111.825)
+		(end 121.55 110.25)
 		(width 0.2)
 		(layer "B.Cu")
@@
 	)
 	(segment
-		(start 119.85 115.025)
-		(end 121.55 113.325)
+		(start 121.55 100.9)
+		(end 124.125 98.325)
 		(width 0.2)
 		(layer "B.Cu")
